File: Microcontroller.kicad_sch (KiCad schematic)
At the start: 17 parts, among them IC3 W25Q128JVSIQ, IC4 ESP32-S3R8, Q1 40MHz

Commit message: test 3
Other:
- note added: "test text"
Changed lines of the file:
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@@
+		)
+	)
+	(text "test text"
+		(exclude_from_sim no)
+		(at 45.72 163.83 0)
+		(effects
+			(font
+				(size 1.27 1.27)
+			)
 		)
 	)
