File: GPIOheaders.kicad_sch (KiCad schematic)
At the start: 10 parts, among them SW1 TS-1010B-B-A, SW2 PTS810SJK250SMTRLFS, SW3 PTS810SJK250SMTRLFS

Commit message: Changes to final schematic
Changed lines of the file:
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@@
 	(text "GPIO Headers"
 		(exclude_from_sim no)
-		(at 59.69 30.48 0)
+		(at 59.69 27.94 0)
 		(effects
 			(font

Commit message: Most of the layout done
Other:
- note added: "Distance between headers - 25.4mm"
- note removed: "Distance between headers - 22.86mm"
Changed lines of the file:
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@@
 		)
 	)
-	(text "Distance between headers - 22.86mm"
+	(text "Distance between headers - 25.4mm"
 		(exclude_from_sim no)
 		(at 60.96 91.44 0)
